File: pcb/projects/micromouse/micromouse.brd (EAGLE design)
At the start: 100 x 80 mm, 44 parts, among them IC1 UA78M33DCY, IC2 UA78M05DCY, M1 332-06, M2 332-06, U1 DSPIC33FJ64MC804-H/PT

Commit message: Add value for resistors for LEDs
Parts:
- R3, R4: value (none) -> 700Ohm
Changed lines of the file:
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@@
 <attribute name="VALUE" x="-88.9" y="-254.635" size="1.27" layer="27"/>
 </element>
-<element name="R3" library="rcl" library_urn="urn:adsk.eagle:library:334" package="R0805" package3d_urn="urn:adsk.eagle:package:23553/2" value="" x="-87.63" y="-259.08" smashed="yes">
+<element name="R3" library="rcl" library_urn="urn:adsk.eagle:library:334" package="R0805" package3d_urn="urn:adsk.eagle:package:23553/2" value="700Ohm" x="-87.63" y="-259.08" smashed="yes">
 <attribute name="NAME" x="-88.265" y="-257.81" size="1.27" layer="25"/>
 <attribute name="POPULARITY" value="86" x="-87.63" y="-259.08" size="1.778" layer="27" display="off"/>
@@
 <attribute name="VALUE" x="-88.265" y="-261.62" size="1.27" layer="27"/>
 </element>
-<element name="R4" library="rcl" library_urn="urn:adsk.eagle:library:334" package="R0805" package3d_urn="urn:adsk.eagle:package:23553/2" value="" x="-87.63" y="-264.16" smashed="yes">
+<element name="R4" library="rcl" library_urn="urn:adsk.eagle:library:334" package="R0805" package3d_urn="urn:adsk.eagle:package:23553/2" value="700Ohm" x="-87.63" y="-264.16" smashed="yes">
 <attribute name="NAME" x="-88.265" y="-262.89" size="1.27" layer="25"/>
 <attribute name="POPULARITY" value="86" x="-87.63" y="-264.16" size="1.778" layer="27" display="off"/>

Commit message: Add solder pad for distance sensor and battery
Parts:
- removed DIST1, DIST2, DIST3: (no value), con-lstb:MA03-1
- added DIST1+, DIST1-, DIST1S, DIST2+, DIST2-, DIST2S, DIST3+, DIST3-, DIST3S, PAD+, PAD-: (no value), wirepad:SMD1,27-2,54
Connections:
- net +5V: now also DIST1+.1, DIST2+.1, DIST3+.1; no longer DIST1.1, DIST2.1, DIST3.1
- net +9V: now also PAD+.1
- net DSENS1: now also DIST1S.1; no longer DIST1.2
- net DSENS2: now also DIST2S.1; no longer DIST2.2
- net DSENS3: now also DIST3S.1; no longer DIST3.2
- net GND: now also DIST1-.1, DIST2-.1, DIST3-.1, PAD-.1; no longer DIST1.3, DIST2.3, DIST3.3
